Commit message: Robot modification

File: my_robot/urdf/my_robot.xacro (robot description, xacro)
@@ -13,10 +13,10 @@
     <pose>0 0 0.1 0 0 0</pose>
     <inertial>
-      <mass value="15.0"/>
+      <mass value="8.0"/>
       <origin xyz="0.0 0 0" rpy=" 0 0 0"/>
       <inertia
-          ixx="0.1" ixy="0" ixz="0"
-          iyy="0.1" iyz="0"
-          izz="0.1"
+          ixx="0.06" ixy="0" ixz="0"
+          iyy="0.06" iyz="0"
+          izz="0.06"
       />
     </inertial>
@@ -24,5 +24,5 @@
       <origin xyz="0 0 0" rpy=" 0 0 0"/>
       <geometry>
-        <box size=".4 .2 .1"/>
+        <box size=".2 .1 .06"/>
       </geometry><link name="camera">
     <collision>
@@ -48,5 +48,5 @@
   <joint name="camera_joint" type="fixed">
     <axis xyz="0 1 0" />
-    <origin xyz=".2 0 0" rpy="0 0 0"/>
+    <origin xyz=".1 0 0" rpy="0 0 0"/>
     <parent link="chassis"/>
     <child link="camera"/>
@@ -56,29 +56,29 @@
       <origin xyz="0 0 0" rpy=" 0 0 0"/>
       <geometry>
-        <box size=".4 .2 .1"/>
+        <box size=".2 .1 .06"/>
       </geometry>
     </visual>
     <collision name='back_caster_collision'>
-      <origin xyz="-0.15 0 -0.05" rpy=" 0 0 0"/>
-      <geometry>
-        <sphere radius="0.0499"/>
+      <origin xyz="-0.07 0 -0.03" rpy=" 0 0 0"/>
+      <geometry>
+        <sphere radius="0.0199"/>
       </geometry>
     </collision>
     <visual name='back_caster_visual'>
-      <origin xyz="-0.15 0 -0.05" rpy=" 0 0 0"/>
-      <geometry>
-        <sphere radius="0.05"/>
+      <origin xyz="-0.07 0 -0.03" rpy=" 0 0 0"/>
+      <geometry>
+        <sphere radius="0.02"/>
       </geometry>
     </visual>
     <collision name='front_caster_collision'>
-      <origin xyz="0.15 0 -0.05" rpy=" 0 0 0"/>
-      <geometry>
-        <sphere radius="0.0499"/>
+      <origin xyz="0.07 0 -0.03" rpy=" 0 0 0"/>
+      <geometry>
+        <sphere radius="0.0199"/>
       </geometry>
     </collision>
     <visual name='front_caster_visual'>
-      <origin xyz="0.15 0 -0.05" rpy=" 0 0 0"/>
-      <geometry>
-        <sphere radius="0.05"/>
+      <origin xyz="0.07 0 -0.03" rpy=" 0 0 0"/>
+      <geometry>
+        <sphere radius="0.02"/>
       </geometry>
     </visual>
@@ -89,5 +89,5 @@
       <origin xyz="0 0 0" rpy="0 1.5707 1.5707"/>
       <geometry>
-        <cylinder radius="0.1" length="0.05"/>
+        <cylinder radius="0.05" length="0.025"/>
       </geometry>
     </collision>
@@ -95,14 +95,14 @@
       <origin xyz="0 0 0" rpy="0 1.5707 1.5707"/>
       <geometry>
-        <cylinder radius="0.1" length="0.05"/>
-      </geometry>
-    </visual>
-    <inertial>
-      <origin xyz="0 0 0" rpy="0 1.5707 1.5707"/>
-      <mass value="5"/>
+        <cylinder radius="0.05" length="0.025"/>
+      </geometry>
+    </visual>
+    <inertial>
+      <origin xyz="0 0 0" rpy="0 1.5707 1.5707"/>
+      <mass value="0.5"/>
       <inertia
-        ixx=".1" ixy="0.0" ixz="0.0"
-        iyy=".1" iyz="0.0"
-        izz=".1"/>
+        ixx=".05" ixy="0.0" ixz="0.0"
+        iyy=".05" iyz="0.0"
+        izz=".05"/>
     </inertial>
   </link>
@@ -112,5 +112,5 @@
       <origin xyz="0 0 0" rpy="0 1.5707 1.5707"/>
       <geometry>
-        <cylinder radius="0.1" length="0.05"/>
+        <cylinder radius="0.05" length="0.025"/>
       </geometry>
     </collision>
@@ -118,18 +118,18 @@
       <origin xyz="0 0 0" rpy="0 1.5707 1.5707"/>
       <geometry>
-        <cylinder radius="0.1" length="0.05"/>
-      </geometry>
-    </visual>
-    <inertial>
-      <origin xyz="0 0 0" rpy="0 1.5707 1.5707"/>
-      <mass value="5"/>
+        <cylinder radius="0.05" length="0.025"/>
+      </geometry>
+    </visual>
+    <inertial>
+      <origin xyz="0 0 0" rpy="0 1.5707 1.5707"/>
+      <mass value="0.5"/>
       <inertia
-        ixx=".1" ixy="0.0" ixz="0.0"
-        iyy=".1" iyz="0.0"
-        izz=".1"/>
+        ixx=".05" ixy="0.0" ixz="0.0"
+        iyy=".05" iyz="0.0"
+        izz=".05"/>
     </inertial>
   </link>
   <joint type="continuous" name="left_wheel_hinge">
-    <origin xyz="0 0.15 0" rpy="0 0 0"/>
+    <origin xyz="0 0.063 0" rpy="0 0 0"/>
     <!--origin xyz="0.1 0.13 0" rpy="0 1.5707 1.5707"/-->
     <child link="left_wheel"/>
@@ -140,5 +140,5 @@
   </joint>
   <joint type="continuous" name="right_wheel_hinge">
-    <origin xyz="0 -0.15 0" rpy="0 0 0"/>
+    <origin xyz="0 -0.063 0" rpy="0 0 0"/>
     <!--origin xyz="0.1 -0.13 0" rpy="0 1.5707 1.5707"/-->
     <child link="right_wheel"/>
@@ -171,5 +171,5 @@
   <joint name="camera_joint" type="fixed">
     <axis xyz="0 1 0" />
-    <origin xyz=".2 0 0" rpy="0 0 0"/>
+    <origin xyz=".1 0 0" rpy="0 0 0"/>
     <parent link="chassis"/>
     <child link="camera"/>
@@ -177,5 +177,5 @@
  <joint name="hokuyo_joint" type="fixed">
     <axis xyz="0 1 0" />
-    <origin xyz=".15 0 .1" rpy="0 0 0"/>
+    <origin xyz=".07 0 .05" rpy="0 0 0"/>
     <parent link="chassis"/>
     <child link="hokuyo"/>

Commit message: Update parameters for smoother navigation

File: my_robot/urdf/my_robot.xacro (robot description, xacro)
@@ -62,5 +62,5 @@
       <origin xyz="-0.07 0 -0.03" rpy=" 0 0 0"/>
       <geometry>
-        <sphere radius="0.0199"/>
+        <sphere radius="0.0198"/>
       </geometry>
     </collision>
@@ -74,5 +74,5 @@
       <origin xyz="0.07 0 -0.03" rpy=" 0 0 0"/>
       <geometry>
-        <sphere radius="0.0199"/>
+        <sphere radius="0.0198"/>
       </geometry>
     </collision>
